File: PendentFront-LED/PendentFront-LED.kicad_sch (KiCad schematic)
At the start: 95 parts, among them J1 Conn_01x03_Pin, J2 Conn_01x02_Pin, U1 74VHC9595FT, U2 74VHC9595FT, U3 74VHC9595FT, U4 74VHC9595FT

Commit message: More routing
Connections:
- net COLOR.BLUE4: now also U3.13 (Q8); no longer U3.9 (Q4)
- net COLOR.RED6: now also U3.9 (Q4); no longer U3.13 (Q8)
Changed lines of the file:
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@@
 	)
 	(bus_entry
+		(at 276.86 152.4)
+		(size 2.54 -2.54)
+		(stroke
+			(width 0)
+			(type default)
+		)
+	)
+	(bus_entry
 		(at 276.86 147.32)
 		(size 2.54 -2.54)
@@
 	)
 	(bus_entry
-		(at 276.86 152.4)
-		(size 2.54 -2.54)
-		(stroke
-			(width 0)
-			(type default)
-		)
-	)
-	(bus_entry
 		(at 276.86 205.74)
 		(size 2.54 -2.54)
@@
 	)
 	(bus_entry
-		(at 276.86 162.56)
-		(size 2.54 -2.54)
-		(stroke
-			(width 0)
-			(type default)
-		)
-	)
-	(bus_entry
 		(at 30.48 144.78)
 		(size -2.54 -2.54)
@@
 	)
 	(bus_entry
+		(at 276.86 162.56)
+		(size 2.54 -2.54)
+		(stroke
+			(width 0)
+			(type default)
+		)
+	)
+	(bus_entry
 		(at 63.5 144.78)
 		(size -2.54 -2.54)
@@
 	(wire
 		(pts
-			(xy 279.4 149.86) (xy 302.26 149.86)
-		)
-		(stroke
-			(width 0)
-			(type default)
-		)
-	)
-	(wire
-		(pts
 			(xy 364.49 66.04) (xy 364.49 63.5)
 		)
@@
 	(wire
 		(pts
+			(xy 279.4 160.02) (xy 302.26 160.02)
+		)
+		(stroke
+			(width 0)
+			(type default)
+		)
+	)
+	(wire
+		(pts
 			(xy 124.46 87.63) (xy 124.46 97.79)
 		)
@@
 	(wire
 		(pts
+			(xy 279.4 149.86) (xy 302.26 149.86)
+		)
+		(stroke
+			(width 0)
+			(type default)
+		)
+	)
+	(wire
+		(pts
 			(xy 49.53 46.99) (xy 49.53 57.15)
 		)
@@
 		)
 	)
+	(bus
+		(pts
+			(xy 276.86 152.4) (xy 276.86 154.94)
+		)
+		(stroke
+			(width 0)
+			(type default)
+		)
+	)
 	(wire
 		(pts
@@
 	(wire
 		(pts
-			(xy 279.4 160.02) (xy 302.26 160.02)
-		)
-		(stroke
-			(width 0)
-			(type default)
-		)
-	)
-	(wire
-		(pts
 			(xy 142.24 87.63) (xy 144.78 87.63)
 		)
@@
 		)
 	)
-	(bus
-		(pts
-			(xy 276.86 152.4) (xy 276.86 154.94)
-		)
-		(stroke
-			(width 0)
-			(type default)
-		)
-	)
 	(wire
 		(pts
@@
 		)
 	)
+	(bus
+		(pts
+			(xy 276.86 162.56) (xy 276.86 187.96)
+		)
+		(stroke
+			(width 0)
+			(type default)
+		)
+	)
 	(wire
 		(pts
@@
 		)
 	)
-	(bus
-		(pts
-			(xy 276.86 162.56) (xy 276.86 187.96)
-		)
-		(stroke
-			(width 0)
-			(type default)
-		)
-	)
 	(wire
 		(pts
@@
 		)
 	)
-	(label "COLOR.BLUE4"
-		(at 302.26 149.86 180)
+	(label "COLOR.BLUE3"
+		(at 68.58 128.27 270)
 		(effects
 			(font
@@
 		)
 	)
-	(label "COLOR.BLUE3"
-		(at 68.58 128.27 270)
+	(label "COLOR.GREEN3"
+		(at 302.26 116.84 180)
 		(effects
 			(font
@@
 		)
 	)
-	(label "COLOR.GREEN3"
-		(at 302.26 116.84 180)
+	(label "COLOR.RED6"
+		(at 302.26 149.86 180)
 		(effects
 			(font
@@
 		)
 	)
-	(label "COLOR.RED6"
-		(at 302.26 160.02 180)
-		(effects
-			(font
-				(size 1.27 1.27)
-			)
-			(justify right bottom)
-		)
-	)
 	(label "COLOR.GREEN3"
 		(at 74.93 128.27 270)
@@
 		(effects
 			(font
+				(size 1.27 1.27)
+			)
+			(justify right bottom)
+		)
+	)
+	(label "COLOR.BLUE4"
+		(at 302.26 160.02 180)
+		(effects
+			(font

Commit message: Nearly done with routing
Connections:
- net ROW1: now also U1.10 (Q5); no longer U1.5 (Q1)
- net ROW2: now also U1.11 (Q6); no longer U1.6 (Q2)
- net ROW3: now also U1.12 (Q7); no longer U1.7 (Q3)
- net ROW4: now also U1.13 (Q8); no longer U1.9 (Q4)
- net ROW5: now also U1.9 (Q4); no longer U1.10 (Q5)
- net ROW6: now also U1.7 (Q3); no longer U1.11 (Q6)
- net ROW7: now also U1.6 (Q2); no longer U1.12 (Q7)
- net ROW8: now also U1.5 (Q1); no longer U1.13 (Q8)
